Commit message: changing the urdf file

File: urdf/brace_top_setup_brace.urdf (robot description, URDF)
Before this commit: robot brace_top_setup_brace, 3 links, 2 joints
Links:
- link Link1: mass 0.09563 -> 0.144521976607446
- link Link2: mass 2.47015 -> 2.41531493094664
- link base_link: mass 0.37798 -> 0.386438799959442
Joints:
- joint Joint1: origin xyz=0 0 -0.025 rpy=0 0 0.523598775598301 -> xyz=-0.0498356367802294 0.00715438320185739 -0.0251410214689495 rpy=0 0 0
- joint Joint2: origin xyz=0 0 -0.365748 rpy=0 0 0 -> xyz=0 0 -0.385747999999974 rpy=0 0 0

Commit message: changing the position of the thigh on the setup to fit reality

File: urdf/brace_top_setup_brace.urdf (robot description, URDF)
Before this commit: robot brace_top_setup_brace, 3 links, 2 joints
Links:
- link Link1: mass 0.144521976607446 -> 0.144521976607445
- link Link2: mass 2.41531493094664 -> 2.4153156910068
Joints:
- joint Joint1: origin xyz=-0.0498356367802294 0.00715438320185739 -0.0251410214689495 rpy=0 0 0 -> xyz=0 0 -0.025 rpy=0 0 0
- joint Joint2: origin xyz=0 0 -0.385747999999974 rpy=0 0 0 -> xyz=0 0 -0.385748000000014 rpy=0 0 0

Commit message: changing the axis for base_link to fit the axis of panda_link8

File: urdf/brace_top_setup_brace.urdf (robot description, URDF)
Before this commit: robot brace_top_setup_brace, 3 links, 2 joints
Links:
- link Link2: mass 2.4153156910068 -> 2.40622270395484
Joints:
- joint Joint1: origin xyz=0 0 -0.025 rpy=0 0 0 -> xyz=0 0 0.0249999999999868 rpy=-3.14159265358979 0 0

Commit message: replacing some 3D printed parts by machined ones

File: urdf/brace_top_setup_brace.urdf (robot description, URDF)
Before this commit: robot brace_top_setup_brace, 3 links, 2 joints
Links:
- link Link2: mass 2.40622270395484 -> 2.33700912012721
- link base_link: mass 0.386438799959442 -> 0.510468252967356
Joints:
- joint Joint1: origin xyz=0 0 0.0249999999999868 rpy=-3.14159265358979 0 0 -> xyz=0 0 0.0256499999999596 rpy=-3.14159265358979 0 0
- joint Joint2: origin xyz=0 0 -0.385748000000014 rpy=0 0 0 -> xyz=0 0 -0.37774800000004 rpy=0 0 0

Commit message: changing the brace assembly to put the new cams and adjust the lenghts of the aluminium tubes

File: urdf/brace_top_setup_brace.urdf (robot description, URDF)
Before this commit: robot brace_top_setup_brace, 3 links, 2 joints
Links:
- link Link2: mass 2.33700912012721 -> 1.86856831514573
Joints:
- joint Joint1: origin xyz=0 0 0.0256499999999596 rpy=-3.14159265358979 0 0 -> xyz=0 0 0.0256500000001189 rpy=-3.14159265358979 0 0
- joint Joint2: origin xyz=0 0 -0.37774800000004 rpy=0 0 0 -> xyz=0 0 -0.377747999999882 rpy=0 0 0

Commit message: correcting error : the brace wasn't included in link2 in the previous commit

File: urdf/brace_top_setup_brace.urdf (robot description, URDF)
Before this commit: robot brace_top_setup_brace, 3 links, 2 joints
Links:
- link Link2: mass 1.86856831514573 -> 2.67816098290905
